Commit message: Closer to reality simulation parameters

File: config/gazebo/models/x340/x340.xacro (robot description, xacro)
@@ -16,8 +16,8 @@
 	<xacro:property name="mass_rotor" value="0.009" /> <!-- [kg] -->
 	<xacro:property name="arm_length" value="0.17" /> <!-- [m] -->
-	<xacro:property name="arm_length_xy" value="0.1202" />
+	<xacro:property name="arm_length_xy" value="0.1202" /> <!-- [m] -->
 	<xacro:property name="rotor_offset_top" value="0.0315" /> <!-- [m] -->
 	<xacro:property name="radius_rotor" value="0.1016" /> <!-- [m] -->
-	<xacro:property name="motor_constant" value="8.54858e-06" /> <!-- [kg m/s^2] -->
+	<xacro:property name="motor_constant" value="5.403546e-06" /> <!-- [kg m/s^2] -->
 	<xacro:property name="moment_constant" value="0.016" /> <!-- [m] -->
 	<xacro:property name="time_constant_up" value="0.0125" /> <!-- [s] -->
