File: hardware/beacon/schematic/shield.brd (EAGLE design)
At the start: 25.4 x 58.9 mm, 10 parts

Commit message: Add more notes and code adjustments
Connections:
- new net DO_NOT_CONNECT: B1.8
- net VBAT_SCAL: now also B1.9; no longer B1.8
Routing:
- net VBAT_SCAL: track 9.67 -> 10.6 mm
Changed lines of the file:
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@@
 </signal>
 <signal name="VBAT_SCAL">
-<contactref element="B1" pad="8"/>
 <contactref element="R3" pad="1"/>
 <contactref element="R2" pad="2"/>
 <wire x1="6.92" y1="15.33" x2="6.98" y2="15.33" width="0.508" layer="1"/>
 <wire x1="6.98" y1="15.33" x2="6.98" y2="19.14" width="0.508" layer="1"/>
-<wire x1="6.98" y1="19.14" x2="1.27" y2="19.14" width="0.508" layer="1"/>
-<wire x1="1.27" y1="19.14" x2="1.27" y2="19.05" width="0.508" layer="1"/>
+<contactref element="B1" pad="9"/>
+<wire x1="6.98" y1="19.14" x2="3.72" y2="19.14" width="0.4064" layer="1"/>
+<wire x1="3.72" y1="19.14" x2="1.27" y2="21.59" width="0.4064" layer="1"/>
 </signal>
 <signal name="VBAT">
@@
 <wire x1="21.59" y1="21.59" x2="24.13" y2="24.13" width="0.508" layer="16"/>
 </signal>
+<signal name="DO_NOT_CONNECT">
+<contactref element="B1" pad="8"/>
+</signal>
 </signals>
