File: hardware/beacon/schematic/shield.sch (EAGLE design)
At the start: 10 parts

Commit message: Add more notes and code adjustments
Connections:
- new net DO_NOT_CONNECT: B1.12
- net VBAT_SCAL: now also B1.14; no longer B1.12
Changed lines of the file:
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@@
 <net name="VBAT_SCAL" class="0">
-<segment>
-<pinref part="B1" gate="G$1" pin="12"/>
-<wire x1="38.1" y1="45.72" x2="15.24" y2="45.72" width="0.1524" layer="91"/>
-<label x="15.24" y="45.72" size="1.778" layer="95"/>
-</segment>
 <segment>
 <pinref part="R3" gate="G$1" pin="1"/>
@@
 <junction x="63.5" y="109.22"/>
 <label x="73.66" y="109.22" size="1.778" layer="95"/>
+</segment>
+<segment>
+<pinref part="B1" gate="G$1" pin="14"/>
+<wire x1="38.1" y1="48.26" x2="15.24" y2="48.26" width="0.1524" layer="91"/>
+<label x="15.24" y="48.26" size="1.778" layer="95"/>
 </segment>
 </net>
@@
 </segment>
 </net>
+<net name="DO_NOT_CONNECT" class="0">
+<segment>
+<pinref part="B1" gate="G$1" pin="12"/>
+<wire x1="38.1" y1="45.72" x2="15.24" y2="45.72" width="0.1524" layer="91"/>
+<label x="15.24" y="45.72" size="1.778" layer="95"/>
+</segment>
+</net>
